File: Platine/HM-ES-PMSw1-Pl_GosundSP1.sch (KiCad schematic (older format))
At the start: 16 parts, among them J1 Conn_BW-SHP2, J2 FTDI, J3 Conn_01x04, J4 Reset, J7 Ant, J8 AntGND, U2 CC1101

Commit message: update schematic
Parts:
- J2: footprint Pin_Headers:Pin_Header_Straight_1x06 -> Pin_Headers:Pin_Header_Straight_1x06_Pitch2.54mm
- U1: renamed from U?; footprint TQFP44 -> Housings_QFP:TQFP-44_10x10mm_Pitch0.8mm
- renumbered C6 to C1, C1 to C2, C2 to C3, C3 to C4, C4 to C5, C5 to C6, C8 to C7
Connections:
- net labels added: D2, D3
- net labels removed: B3, RXD, TXD
- wire segments 74 -> 82
- no-connect marks 6 -> 24
Other:
- note added: "CF1\nButton\nLED red\n\nRX\nVCC"
- note added: "EN"
- note added: "SEL\nRelay\nLED blue\nCF\nTX\nGND"
- note added: "tout"
- note removed: "EN\nCF1\nButton\nLED red\n?\nRX\nVCC"
- note removed: "tout\nSEL\nRelay\nLED blue\nCF\nTX\nGND"

Commit message: oard V0.1 routing complete
Parts:
- removed J7: Ant, Connectors:Pin_d0.7mm_L6.5mm_W1.8mm_FlatFork, symbol Conn_01x01
- removed J8: AntGND, Connectors:Pin_d0.7mm_L6.5mm_W1.8mm_FlatFork, symbol Conn_01x01
- J4: footprint Connectors:Pin_d0.7mm_L6.5mm_W1.8mm_FlatFork -> SMD_Packages:1Pin
- U2: footprint CC1101_Module:CC1101_Module -> CC1101_Module:CC1101_SMD
Connections:
- net labels added: BUTTON, CF, CF1, GDO0, LED_blue, LED_red, RELAY, SEL
- net labels removed: B0, B1, B2, D2, D3, D5, D6, D7
- wire segments 82 -> 81
- no-connect marks 24 -> 25
Changed lines of the file:
@@
 F 0 "U2" H 9250 2875 60  0000 C CNN
 F 1 "CC1101" H 9250 1875 60  0000 C CNN
-F 2 "CC1101_Module:CC1101_Module" H 9100 2925 60  0001 C CNN
+F 2 "CC1101_Module:CC1101_SMD" H 9100 2925 60  0001 C CNN
 F 3 "" H 9100 2925 60  0001 C CNN
 	1    9250 2375
@@
 Text Label 1625 6275 0    60   ~ 0
 Reset
-$Comp
-L Conn_01x01 J7
-U 1 1 5AD41019
-P 10250 2375
-F 0 "J7" H 10400 2375 50  0000 C CNN
-F 1 "Ant" H 10550 2375 50  0000 C CNN
-F 2 "Connectors:Pin_d0.7mm_L6.5mm_W1.8mm_FlatFork" H 10250 2375 50  0001 C CNN
-F 3 "" H 10250 2375 50  0001 C CNN
-	1    10250 2375
-	1    0    0    -1
-$EndComp
-$Comp
-L Conn_01x01 J8
-U 1 1 5ADF8BE1
-P 10250 2525
-F 0 "J8" H 10400 2525 50  0000 C CNN
-F 1 "AntGND" H 10625 2525 50  0000 C CNN
-F 2 "Connectors:Pin_d0.7mm_L6.5mm_W1.8mm_FlatFork" H 10250 2525 50  0001 C CNN
-F 3 "" H 10250 2525 50  0001 C CNN
-	1    10250 2525
-	1    0    0    -1
-$EndComp
 Text Notes 850  4475 0    60   ~ 0
 FTDI
@@
 F 0 "J4" H 1250 3550 50  0000 C CNN
 F 1 "Reset" H 1400 3550 50  0000 C CNN
-F 2 "Connectors:Pin_d0.7mm_L6.5mm_W1.8mm_FlatFork" H 1100 3550 50  0001 C CNN
+F 2 "SMD_Packages:1Pin" H 1100 3550 50  0001 C CNN
 F 3 "" H 1100 3550 50  0001 C CNN
 	1    1100 3550
@@
 L VCC #PWR012
 U 1 1 5B8AAF2B
-P 9275 5000
-F 0 "#PWR012" H 9275 4850 50  0001 C CNN
-F 1 "VCC" H 9275 5150 50  0000 C CNN
-F 2 "" H 9275 5000 50  0001 C CNN
-F 3 "" H 9275 5000 50  0001 C CNN
-	1    9275 5000
+P 9425 5000
+F 0 "#PWR012" H 9425 4850 50  0001 C CNN
+F 1 "VCC" H 9425 5150 50  0000 C CNN
+F 2 "" H 9425 5000 50  0001 C CNN
+F 3 "" H 9425 5000 50  0001 C CNN
+	1    9425 5000
 	1    0    0    -1
 $EndComp
@@
 Text Notes 9900 5000 0    60   ~ 0
 CF1\nButton\nLED red\n\nRX\nVCC
-Text Label 9150 4600 2    60   ~ 0
-D5
-Text Label 8250 4600 0    60   ~ 0
-B1
+Text Label 9300 4600 2    60   ~ 0
+BUTTON
+Text Label 8050 4600 0    60   ~ 0
+RELAY
 NoConn ~ 8450 4400
 NoConn ~ 8950 4800
-Text Label 8250 4700 0    60   ~ 0
-B0
-Text Label 9150 4700 2    60   ~ 0
-D7
-Text Label 8250 4800 0    60   ~ 0
-D3
-Text Label 9150 4500 2    60   ~ 0
-B2
-Text Label 8250 4500 0    60   ~ 0
-D6
+Text Label 8050 4700 0    60   ~ 0
+LED_blue
+Text Label 9300 4700 2    60   ~ 0
+LED_red
+Text Label 8050 4800 0    60   ~ 0
+CF
+Text Label 9300 4500 2    60   ~ 0
+CF1
+Text Label 8050 4500 0    60   ~ 0
+SEL
 $Comp
 L ATMEGA644PA-AU U1
@@
 Wire Wire Line
 	9975 2225 9975 2650
-Wire Wire Line
-	9800 2525 10050 2525
 Connection ~ 9975 2525
 Wire Wire Line
@@
 	1325 6275 1625 6275
 Wire Wire Line
-	10050 2375 9800 2375
-Wire Wire Line
 	1325 4750 1450 4750
 Wire Wire Line
@@
 	8250 5000 8250 5050
 Wire Wire Line
-	8450 4800 8250 4800
-Wire Wire Line
-	8250 4700 8450 4700
-Wire Wire Line
-	8450 4600 8250 4600
-Wire Wire Line
-	8450 4500 8250 4500
-Wire Wire Line
-	8950 4500 9150 4500
-Wire Wire Line
-	8950 4600 9150 4600
-Wire Wire Line
-	8950 4700 9150 4700
-Wire Wire Line
-	9275 5000 8950 5000
+	8450 4800 8050 4800
+Wire Wire Line
+	8050 4700 8450 4700
+Wire Wire Line
+	8450 4600 8050 4600
+Wire Wire Line
+	8450 4500 8050 4500
+Wire Wire Line
+	8950 4500 9300 4500
+Wire Wire Line
+	8950 4600 9300 4600
+Wire Wire Line
+	8950 4700 9300 4700
+Wire Wire Line
+	9425 5000 8950 5000
 Wire Wire Line
 	4850 975  4850 1150
@@
 RESET
 Wire Wire Line
-	6150 2850 6350 2850
-Wire Wire Line
-	6150 2950 6350 2950
-Wire Wire Line
-	6150 3050 6350 3050
-Wire Wire Line
-	6150 2750 6350 2750
+	6150 2850 6550 2850
+Wire Wire Line
+	6150 2950 6550 2950
+Wire Wire Line
+	6150 3050 6550 3050
+Wire Wire Line
+	6150 2750 6550 2750
 Wire Wire Line
 	8500 2225 8750 2225
@@
 Text Label 8500 2725 0    60   ~ 0
 CS
-Text Label 6350 2750 2    60   ~ 0
+Text Label 6550 2750 2    60   ~ 0
 CS
-Text Label 6350 2850 2    60   ~ 0
+Text Label 6550 2850 2    60   ~ 0
 MOSI
-Text Label 6350 2950 2    60   ~ 0
+Text Label 6550 2950 2    60   ~ 0
 MISO
-Text Label 6350 3050 2    60   ~ 0
+Text Label 6550 3050 2    60   ~ 0
 SCK
 Text Notes 1175 4300 0    60   Italic 12
 DNI
-Wire Wire Line
-	6150 2450 6350 2450
 NoConn ~ 8950 4400
 Wire Wire Line
-	8250 4900 8450 4900
-Wire Wire Line
-	8950 4900 9150 4900
-Text Label 8250 4900 0    60   ~ 0
+	8050 4900 8450 4900
+Wire Wire Line
+	8950 4900 9300 4900
+Text Label 8050 4900 0    60   ~ 0
 TX
-Text Label 9150 4900 2    60   ~ 0
+Text Label 9300 4900 2    60   ~ 0
 RX
 Wire Wire Line
-	6150 2550 6350 2550
-Wire Wire Line
-	6150 4650 6350 4650
-Wire Wire Line
-	6150 4750 6350 4750
-Text Label 6350 2450 2    60   ~ 0
-B1
-Text Label 6350 2550 2    60   ~ 0
-B2
-Text Label 6350 4650 2    60   ~ 0
-D5
-Text Label 6350 4750 2    60   ~ 0
-D6
+	6150 2550 6550 2550
+Wire Wire Line
+	6150 4650 6550 4650
+Wire Wire Line
+	6150 4750 6550 4750
+Text Label 6550 2550 2    60   ~ 0
+GDO0
+Text Label 6550 4650 2    60   ~ 0
+BUTTON
+Text Label 6550 4750 2    60   ~ 0
+LED_blue
 Text Notes 9500 5450 0    60   ~ 0
 red LED: on/off state\nblue LED: connection indication
 Wire Wire Line
-	6150 2350 6350 2350
-Text Label 6350 2350 2    60   ~ 0
-B0
-Wire Wire Line
-	6150 4850 6350 4850
-Text Label 6350 4850 2    60   ~ 0
-D7
+	6150 4850 6550 4850
+Text Label 6550 4850 2    60   ~ 0
+LED_red
 $Comp
 L C C4
@@
 Oct. 2018
 Text Label 8500 2625 0    60   ~ 0
-D2
-Wire Wire Line
-	6150 4150 6350 4150
-Text Label 6350 4350 2    60   ~ 0
-D2
+GDO0
+Wire Wire Line
+	6150 4150 6550 4150
+Text Label 6550 4350 2    60   ~ 0
+CF1
 $Comp
 L GND #PWR018
@@
 $EndComp
 Wire Wire Line
-	4950 5350 4950 5150
+	4950 5150 4950 5350
 Wire Wire Line
 	4850 5150 4850 5275
@@
 Connection ~ 5050 5275
 Wire Wire Line
-	6150 4250 6350 4250
-Wire Wire Line
-	6150 4350 6350 4350
-Text Label 6350 4150 2    60   ~ 0
+	6150 4250 6550 4250
+Wire Wire Line
+	6150 4350 6550 4350
+Text Label 6550 4150 2    60   ~ 0
 RX
-Text Label 6350 4250 2    60   ~ 0
+Text Label 6550 4250 2    60   ~ 0
 TX
 Wire Wire Line
-	6150 4450 6350 4450
-Text Label 6350 4450 2    60   ~ 0
-D3
+	6150 4450 6550 4450
+Text Label 6550 4450 2    60   ~ 0
+CF
 Wire Notes Line
 	9875 4325 9875 5025
@@
 NoConn ~ 6150 2150
 NoConn ~ 6150 3250
-NoConn ~ 6150 3350
 NoConn ~ 6150 3450
 NoConn ~ 6150 3550
@@
 NoConn ~ 6150 3850
 NoConn ~ 6150 3950
-NoConn ~ 6150 4550
 NoConn ~ 6150 2650
+Wire Wire Line
+	6150 4550 6550 4550
+Text Label 6550 4550 2    60   ~ 0
+RELAY
+Wire Wire Line
+	6150 3350 6550 3350
+Text Label 6550 3350 2    60   ~ 0
+SEL
+NoConn ~ 6150 2350
+NoConn ~ 6150 2450
+Wire Wire Line
+	9800 2525 9975 2525
+NoConn ~ 9800 2375
 $EndSCHEMATC

Commit message: add resonator for better clock
e.g. CSTCE8M00G55-R0, available at Reichelt (CSTCE 8,00)
Parts:
- added R2: 1M, Resistors_SMD:R_0603_HandSoldering, symbol R
- added Y1: Resonator, Resonators:Resonator_SMD_muRata_TPSKA-3pin_7.9x3.8mm_HandSoldering, symbol Resonator
Connections:
- wire segments 81 -> 89
- no-connect marks 25 -> 23
Other:
- note added: "1.0"
- note removed: "0.1"
Changed lines of the file:
@@
 $EndComp
 Text Notes 10575 7650 0    60   ~ 0
-0.1
+1.0
 $Comp
 L VCC #PWR010
@@
 	1    0    0    -1
 $EndComp
-NoConn ~ 4150 2250
-NoConn ~ 4150 1850
 Wire Wire Line
 	1350 2975 1350 3125
@@
 	9800 2525 9975 2525
 NoConn ~ 9800 2375
+$Comp
+L Resonator Y1
+U 1 1 5BDC373F
+P 3800 2050
+F 0 "Y1" H 3800 2275 50  0000 C CNN
+F 1 "Resonator" H 3800 2200 50  0000 C CNN
+F 2 "Resonators:Resonator_SMD_muRata_TPSKA-3pin_7.9x3.8mm_HandSoldering" H 3775 2050 50  0001 C CNN
+F 3 "" H 3775 2050 50  0001 C CNN
+	1    3800 2050
+	0    1    1    0
+$EndComp
+Wire Wire Line
+	3800 1900 3800 1850
+Wire Wire Line
+	3400 1850 4150 1850
+Wire Wire Line
+	3800 2200 3800 2250
+Wire Wire Line
+	3400 2250 4150 2250
+$Comp
+L R R2
+U 1 1 5BDC3B63
+P 3400 2050
+F 0 "R2" V 3480 2050 50  0000 C CNN
+F 1 "1M" V 3400 2050 50  0000 C CNN
+F 2 "Resistors_SMD:R_0603_HandSoldering" V 3330 2050 50  0001 C CNN
+F 3 "" H 3400 2050 50  0001 C CNN
+	1    3400 2050
+	1    0    0    -1
+$EndComp
+Wire Wire Line
+	3400 1900 3400 1850
+Connection ~ 3800 1850
+Wire Wire Line
+	3400 2200 3400 2250
+Connection ~ 3800 2250
+$Comp
+L GND #PWR019
+U 1 1 5BDC3CD4
+P 3550 2350
+F 0 "#PWR019" H 3550 2100 50  0001 C CNN
+F 1 "GND" H 3550 2200 50  0000 C CNN
+F 2 "" H 3550 2350 50  0001 C CNN
+F 3 "" H 3550 2350 50  0001 C CNN
+	1    3550 2350
+	1    0    0    -1
+$EndComp
+Wire Wire Line
+	3600 2050 3550 2050
+Wire Wire Line
+	3550 2050 3550 2350
+Text Notes 1600 3100 0    60   Italic 12
+DNI
+Text Notes 700  3500 0    60   Italic 12
+DNI
 $EndSCHEMATC

Commit message: finalize V1.0
fix #1, #2, #4
Parts:
- J4: footprint SMD_Packages:1Pin -> Testpads:Testpad
Changed lines of the file:
@@
 F 0 "J4" H 1250 3550 50  0000 C CNN
 F 1 "Reset" H 1400 3550 50  0000 C CNN
-F 2 "SMD_Packages:1Pin" H 1100 3550 50  0001 C CNN
+F 2 "Testpads:Testpad" H 1100 3550 50  0001 C CNN
 F 3 "" H 1100 3550 50  0001 C CNN
 	1    1100 3550

Commit message: Support for Gosund SP1 V2.3 (new WiFi module)
Parts:
- removed J1: Conn_BW-SHP2, BW-SHP2:BW-SHP2-Con, symbol Conn_02x07_Odd_Even
- added J11: BW_Gosund_Con, BW-SHP2:Gosund_SP1-C_V2.3, symbol BW_Gosund_Con
Connections:
- no-connect marks 23 -> 20
Changed lines of the file:
@@
 LIBS:valves
 LIBS:cc1101-module
+LIBS:BW_Gosund_Con
 LIBS:HM-ES-PMSw1-Pl_GosundSP1-cache
 EELAYER 25 0
@@
 $EndComp
 $Comp
-L Conn_02x07_Odd_Even J1
-U 1 1 5B8AAF58
-P 8650 4700
-F 0 "J1" H 8700 5100 50  0000 C CNN
-F 1 "Conn_BW-SHP2" H 8700 4300 50  0000 C CNN
-F 2 "BW-SHP2:BW-SHP2-Con" H 8650 4700 50  0001 C CNN
-F 3 "" H 8650 4700 50  0001 C CNN
-	1    8650 4700
-	1    0    0    -1
-$EndComp
-$Comp
 L GND #PWR013
 U 1 1 5B8ABA1A
-P 8250 5050
-F 0 "#PWR013" H 8250 4800 50  0001 C CNN
-F 1 "GND" H 8250 4900 50  0000 C CNN
-F 2 "" H 8250 5050 50  0001 C CNN
-F 3 "" H 8250 5050 50  0001 C CNN
-	1    8250 5050
+P 7950 5050
+F 0 "#PWR013" H 7950 4800 50  0001 C CNN
+F 1 "GND" H 7950 4900 50  0000 C CNN
+F 2 "" H 7950 5050 50  0001 C CNN
+F 3 "" H 7950 5050 50  0001 C CNN
+	1    7950 5050
 	1    0    0    -1
 $EndComp
@@
 Text Label 9300 4600 2    60   ~ 0
 BUTTON
-Text Label 8050 4600 0    60   ~ 0
+Text Label 7750 4600 0    60   ~ 0
 RELAY
-NoConn ~ 8450 4400
-NoConn ~ 8950 4800
-Text Label 8050 4700 0    60   ~ 0
+Text Label 7750 4700 0    60   ~ 0
 LED_blue
 Text Label 9300 4700 2    60   ~ 0
 LED_red
-Text Label 8050 4800 0    60   ~ 0
+Text Label 7750 4800 0    60   ~ 0
 CF
 Text Label 9300 4500 2    60   ~ 0
 CF1
-Text Label 8050 4500 0    60   ~ 0
+Text Label 7750 4500 0    60   ~ 0
 SEL
 $Comp
@@
 Connection ~ 1475 1375
 Wire Wire Line
-	8450 5000 8250 5000
-Wire Wire Line
-	8250 5000 8250 5050
-Wire Wire Line
-	8450 4800 8050 4800
-Wire Wire Line
-	8050 4700 8450 4700
-Wire Wire Line
-	8450 4600 8050 4600
-Wire Wire Line
-	8450 4500 8050 4500
+	8150 5000 7950 5000
+Wire Wire Line
+	7950 5000 7950 5050
+Wire Wire Line
+	8150 4800 7750 4800
+Wire Wire Line
+	7750 4700 8150 4700
+Wire Wire Line
+	8150 4600 7750 4600
+Wire Wire Line
+	8150 4500 7750 4500
 Wire Wire Line
 	8950 4500 9300 4500
@@
 Text Notes 1175 4300 0    60   Italic 12
 DNI
-NoConn ~ 8950 4400
-Wire Wire Line
-	8050 4900 8450 4900
+Wire Wire Line
+	7750 4900 8150 4900
 Wire Wire Line
 	8950 4900 9300 4900
-Text Label 8050 4900 0    60   ~ 0
+Text Label 7750 4900 0    60   ~ 0
 TX
 Text Label 9300 4900 2    60   ~ 0
@@
 Text Notes 700  3500 0    60   Italic 12
 DNI
+$Comp
+L BW_Gosund_Con J11
+U 1 1 5C1D302E
+P 8500 4700
+F 0 "J11" H 8550 5100 50  0000 C CNN
+F 1 "BW_Gosund_Con" H 8550 4300 50  0000 C CNN
+F 2 "BW-SHP2:Gosund_SP1-C_V2.3" H 8500 4700 50  0001 C CNN
+F 3 "" H 8500 4700 50  0001 C CNN
+	1    8500 4700
+	1    0    0    -1
+$EndComp
 $EndSCHEMATC
